File: corne-cherry/pcb/corne-cherry.kicad_sch (KiCad schematic)
At the start: 146 parts, among them J1 MJ-4PP-9, J2 OLED, J3 MJ-4PP-9, J4 OLED, SW1 SW_PUSH, SW10 SW_PUSH, SW11 SW_PUSH, SW12 SW_PUSH, SW13 SW_PUSH, SW14 SW_PUSH, SW15 SW_PUSH, SW16 SW_PUSH, SW17 SW_PUSH, SW18 SW_PUSH, SW19 SW_PUSH, SW2 SW_PUSH, SW20 SW_PUSH, SW21 SW_PUSH, SW22 SW_PUSH, SW23 SW_PUSH, SW24 SW_PUSH, SW25 SW_PUSH, SW26 SW_PUSH, SW27 SW_PUSH, SW28 SW_PUSH, SW29 SW_PUSH, SW3 SW_PUSH, SW30 SW_PUSH, SW31 SW_PUSH, SW32 SW_PUSH, SW33 SW_PUSH, SW34 SW_PUSH, SW35 SW_PUSH, SW36 SW_PUSH, SW37 SW_PUSH, SW38 SW_PUSH, SW39 SW_PUSH, SW4 SW_PUSH, SW40 SW_PUSH, SW41 SW_PUSH, SW42 SW_PUSH, SW5 SW_PUSH, SW6 SW_PUSH, SW7 SW_PUSH, SW8 SW_PUSH, SW9 SW_PUSH, U1 ProMicro, U2 ProMicro

Commit message: Stashing
Parts:
- removed J2, J4: OLED, kbd:OLED_1side, symbol Connector_Generic:Conn_01x04
- removed LED1, LED2, LED28, LED29, LED3, LED30, LED31, LED32, LED33, LED4, LED5, LED6: WS2812B, LED_SMD:LED_WS2812B_PLCC4_5.0x5.0mm_P3.2mm, symbol LED:WS2812B
- removed LED10, LED11, LED12, LED13, LED14, LED15, LED16, LED17, LED18, LED19, LED20, LED21, LED22, LED23, LED24, LED25, LED26, LED27, LED34, LED35, LED36, LED37, LED38, LED39, LED40, LED41, LED42, LED43, LED44, LED45, LED46, LED47, LED48, LED49, LED50, LED51, LED52, LED53, LED54, LED7, LED8, LED9: YS-SK6812MINI-E, kbd:YS-SK6812MINI-E, symbol kbd:YS-SK6812MINI-E
- added C1, C2: C_Small, Resistor SMD:R_0201_0603Metric_Pad0.64x0.40mm_HandSolder, symbol Device:C_Small
- added D43: D, Library:TH 1N4148 Diode (long), symbol Device:D
- added J2: 30 pin Display Connector, Amphenol F3311A7H121030E200:AMPHENOL_F3311A7H121030E200, symbol F3311A7H121030E200:F3311A7H121030E200
- added R1: R, Resistor SMD:R_0603_1608Metric_Pad0.98x0.95mm_HandSolder, symbol Device:R
- added SW43: SW_PUSH, Switch_Keyboard_Hotswap_Kailh:SW_Hotswap_Kailh_Choc_V2_1.00u, symbol kbd:SW_PUSH
- D1, D10, D11, D12, D13, D14, D15, D16, D17, D18, D19, D2, D20, D21, D22, D23, D24, D25, D26, D27, D28, D29, D3, D30, D31, D32, D33, D34, D35, D36, D37, D38, D39, D4, D40, D41, D42, D5, D6, D7, D8, D9: footprint kbd:D3_SMD_v2 -> Library:TH 1N4148 Diode (long)
- J1, J3: footprint kbd:MJ-4PP-9_1side -> kbd:MJ-4PP-9
- RSW1, RSW2: footprint kbd:ResetSW_1side -> kbd:ResetSW
- SW1, SW10, SW11, SW12, SW13, SW14, SW15, SW16, SW17, SW18, SW19, SW2, SW20, SW22, SW23, SW24, SW25, SW26, SW27, SW28, SW29, SW3, SW30, SW31, SW32, SW33, SW34, SW35, SW36, SW37, SW38, SW39, SW4, SW40, SW41, SW5, SW6, SW7, SW8, SW9: footprint kbd:CherryMX_Hotswap -> Switch_Keyboard_Hotswap_Kailh:SW_Hotswap_Kailh_Choc_V2_1.00u
- SW21, SW42: footprint kbd:CherryMX_Hotswap_1.5u -> Switch_Keyboard_Hotswap_Kailh:SW_Hotswap_Kailh_Choc_V2_1.50u
- U1: footprint kbd:ProMicro_v3 -> marbastlib-xp-promicroish:Helios_AC; symbol kbd:ProMicro -> marbastlib-promicroish:Helios; now left out of the parts list
- U2: footprint kbd:ProMicro_v3 -> marbastlib-xp-promicroish:Helios_AC
Connections:
- net GND: now also U1.14 (GND), C1.1, C2.1, J2.1 (GND), J2.11 (D0), J2.12 (D1), J2.13 (D3), J2.14 (D4), J2.15 (D5), J2.16 (D6), J2.17 (D7), J2.18 (D8), J2.25 (GND), J2.30 (GND), J2.9 (RD), R1.1; no longer U1.23 (GND)
- net SDA: now also J2.10 (SDA)
- net VCC: now also U1.16 (3V3), C1.2, C2.2, J2.2 (VCC), J2.20 (LEDA), J2.3 (IM2), J2.4 (IM1); no longer U1.21 (VCC)
- net col0: now also U1.17 (P29); no longer U1.20 (F4/A3)
- net col1: now also U1.18 (P28); no longer U1.19 (F5/A2)
- net col2: now also U1.28 (P15), SW43.1; no longer U1.18 (F6/A1)
- net col3: now also U1.29 (P16); no longer U1.17 (F7/A0)
- net col4: now also U1.11 (P8); no longer U1.16 (B1/15)
- net col5: now also U1.12 (P9); no longer U1.15 (B3/14)
- net reset: now also U1.15 (RST), J2.5 (RST); no longer U1.22 (RST)
- net row3: now also D43.1 (K)
- net SPI_CS: now reaches U1.24 (P21)
- net LED: no longer names the net of U1.1 (P0)
- new net: D43.2 (A), SW43.2
- new net: J2.21 (LEDK), J2.22 (LEDK), J2.23 (LEDK), J2.24 (LEDK), R1.2
- new net GPIO_AD1: U1.20 (P26)
- new net GPIO_AD2: J2.6 (CS), U1.19 (P27)
- new net MISO: U1.22 (P20)
- new net MOSI: J2.8 (SPI-RS), U1.23 (P23)
- new net SCLK: J2.7 (SCL), U1.21 (P22)
- no-connect marks 14 -> 22
Other:
- moved on the sheet: J1, RSW1
