File: sandevistan42/pcb/sandevistan44_left.kicad_pcb (KiCad board)
At the start: 2 copper layers, 354 x 110 mm, 113 parts, among them J1 TRRS, J2 TRRS, SW1 SW_PUSH, SW10 SW_PUSH, SW11 SW_PUSH, SW12 SW_PUSH, SW13 SW_PUSH, SW14 SW_PUSH, SW15 SW_PUSH, SW16 SW_PUSH, SW17 SW_PUSH, SW18 SW_PUSH, SW19 SW_PUSH, SW2 SW_PUSH, SW20 SW_PUSH, SW21 SW_PUSH, SW22 SW_PUSH, SW23 SW_PUSH, SW24 SW_PUSH, SW25 SW_PUSH, SW26 SW_PUSH, SW27 SW_PUSH, SW28 SW_PUSH, SW29 SW_PUSH, SW3 SW_PUSH, SW30 SW_PUSH, SW31 SW_PUSH, SW32 SW_PUSH, SW33 SW_PUSH, SW34 SW_PUSH, SW35 SW_PUSH, SW36 SW_PUSH, SW37 SW_PUSH, SW38 SW_PUSH, SW39 SW_PUSH, SW4 SW_PUSH, SW40 SW_PUSH, SW41 SW_PUSH, SW42 SW_PUSH, SW43 SW_PUSH, SW44 SW_PUSH, SW5 SW_PUSH, SW6 SW_PUSH, SW7 SW_PUSH, SW8 SW_PUSH, SW9 SW_PUSH, U1 ProMicro, U2 ProMicro

Commit message: Split pcbs into separate files and add plates
Parts:
- removed D23, D24, D25, D26, D27, D28, D29, D30, D31, D32, D33, D34, D35, D36, D37, D38, D39, D40, D41, D42, D43, D44: D, Library:TH 1N4148 Diode (long)
- removed J2: TRRS, SJ2 35954A SMT TR:CUI_SJ2-35954A-SMT-TR
- removed J3: ~, vik:vik-keyboard-connector-horizontal
- removed MB1, MB2: ~, Library:3-Pole Mouse Switch
- removed OLED1: 757-NHD-1.91-176176UBC3-ND, Library:NHD-1.91-176176UBC3
- removed RSW2: SW_PUSH, kbd:ResetSW
- removed the Ref** at (204.2, -163.0)
- removed the Ref** at (276.7, -196.2)
- removed the Ref** at (170.1, -136.1)
- removed the Ref** at (181.1, -211.9)
- removed the Ref** at (276.7, -211.9)
- removed the Ref** at (236.7, -136.1)
- removed SW23, SW24, SW25, SW26, SW27, SW28, SW29, SW30, SW31, SW32, SW33, SW34, SW35, SW36, SW37, SW38, SW39, SW40, SW41, SW42, SW43: SW_PUSH, Library:SW_Hotswap_Kailh_Choc_V2_1.00u
- removed SW44: SW_PUSH, Library:SW_Hotswap_Kailh_Choc_V2_1.25u
- removed U2: ProMicro, marbastlib-xp-promicroish:Helios_AC
- added DISP1: DFR0664, Library:DFR0664_2in_RGB_TFT_Display_3_standoff, F.Cu at (177.1, 102.6)
- RESET: renamed from RSW1; footprint kbd:ResetSW -> TL6340AF160Q:SW_TL6340AF160Q
- moved D1 297.6 mm to (79.1, 59.3)
- moved D15 297.6 mm to (138.5, 52.8)
- moved D17 297.6 mm to (144.7, 50.3)
- moved D20 297.6 mm to (160.1, 51.3)
- moved D21 297.6 mm to (164.5, 51.4)
- moved D3 297.6 mm to (83.4, 55.1)
- moved D5 297.6 mm to (95.0, 57.1)
- moved D6 297.6 mm to (94.9, 52.9)
- moved D7 297.6 mm to (104.7, 56.7)
- moved D8 297.6 mm to (105.5, 53.1)
- moved D9 297.6 mm to (109.8, 53.1)
- moved Ref** 297.6 mm to (183.0, 123.7)
- moved Ref** 297.6 mm to (76.4, 63.6)
- moved Ref** 297.6 mm to (116.4, 123.7)
- moved Ref** 297.6 mm to (172.0, 47.9)
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Routing:
- net col0_r: track 152.2 -> 0.00 mm, vias 4 -> 0
- net col4_r: track 146.8 -> 0.00 mm, vias 6 -> 0
- net col2_r: track 141.0 -> 0.00 mm, vias 5 -> 0
- net col1_r: track 134.8 -> 0.00 mm, vias 6 -> 0
- net col3_r: track 121.6 -> 0.00 mm, vias 5 -> 0
- net col5_r: track 102.2 -> 0.00 mm, vias 6 -> 0
- net GND_r: track 101.7 -> 0.00 mm, vias 7 -> 0
- net VCC_r: track 97.8 -> 0.00 mm, vias 5 -> 0
- net GND: track 28.7 -> 114.0 mm, vias 1 -> 6
- net reset: track 0.00 -> 74.3 mm, vias 0 -> 3
- net SDA_r: track 62.0 -> 0.00 mm, vias 3 -> 0
- net RAW_r: track 61.0 -> 0.00 mm, vias 3 -> 0
- net SCL_r: track 59.4 -> 0.00 mm, vias 3 -> 0
- net data: track 85.9 -> 33.6 mm
- net VCC: track 108.2 -> 61.1 mm
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Other:
- board size 354 x 110 mm -> 153.7 x 110 mm
