File: sandevistan42/pcb/sandevistan44_left_plate.kicad_pcb (KiCad board)
At the start: 2 copper layers, 354 x 110 mm, 113 parts, among them J1 TRRS, J2 TRRS, SW1 SW_PUSH, SW10 SW_PUSH, SW11 SW_PUSH, SW12 SW_PUSH, SW13 SW_PUSH, SW14 SW_PUSH, SW15 SW_PUSH, SW16 SW_PUSH, SW17 SW_PUSH, SW18 SW_PUSH, SW19 SW_PUSH, SW2 SW_PUSH, SW20 SW_PUSH, SW21 SW_PUSH, SW22 SW_PUSH, SW23 SW_PUSH, SW24 SW_PUSH, SW25 SW_PUSH, SW26 SW_PUSH, SW27 SW_PUSH, SW28 SW_PUSH, SW29 SW_PUSH, SW3 SW_PUSH, SW30 SW_PUSH, SW31 SW_PUSH, SW32 SW_PUSH, SW33 SW_PUSH, SW34 SW_PUSH, SW35 SW_PUSH, SW36 SW_PUSH, SW37 SW_PUSH, SW38 SW_PUSH, SW39 SW_PUSH, SW4 SW_PUSH, SW40 SW_PUSH, SW41 SW_PUSH, SW42 SW_PUSH, SW43 SW_PUSH, SW44 SW_PUSH, SW5 SW_PUSH, SW6 SW_PUSH, SW7 SW_PUSH, SW8 SW_PUSH, SW9 SW_PUSH, U1 ProMicro, U2 ProMicro

Commit message: Split pcbs into separate files and add plates
Parts:
- removed D1, D10, D11, D12, D13, D14, D15, D16, D17, D18, D19, D2, D20, D21, D22, D23, D24, D25, D26, D27, D28, D29, D3, D30, D31, D32, D33, D34, D35, D36, D37, D38, D39, D4, D40, D41, D42, D43, D44, D5, D6, D7, D8, D9: D, Library:TH 1N4148 Diode (long)
- removed J1, J2: TRRS, SJ2 35954A SMT TR:CUI_SJ2-35954A-SMT-TR
- removed MBIO1: F3311A7H121004E200, Amphenol Footprint Symbol:AMPHENOL_F3311A7H121004E200
- removed OLED1: 757-NHD-1.91-176176UBC3-ND, Library:NHD-1.91-176176UBC3_3_standoff
- removed RSW1, RSW2: SW_PUSH, kbd:ResetSW
- removed Ref** (x14): Val**, Mounting Hole:MountingHole_2.2mm_M2_DIN965
- removed Ref** (x2): 95.5931, Mounting Hole:MountingHole_2.2mm_M2_DIN965
- removed SW1, SW10, SW11, SW12, SW13, SW14, SW15, SW16, SW17, SW18, SW19, SW2, SW20, SW21, SW23, SW24, SW25, SW26, SW27, SW28, SW29, SW3, SW30, SW31, SW32, SW33, SW34, SW35, SW36, SW37, SW38, SW39, SW4, SW40, SW41, SW42, SW43, SW5, SW6, SW7, SW8, SW9: SW_PUSH, Library:SW_Hotswap_Kailh_Choc_V2_1.00u
- removed SW22, SW44: SW_PUSH, Library:SW_Hotswap_Kailh_Choc_V2_1.25u
- removed U1, U2: ProMicro, marbastlib-xp-promicroish:Helios_AC
- removed VIK1: ~, vik:vik-keyboard-connector-horizontal-mini
- added G***: LOGO, Library:logo_ascii_large, B.Cu at (186.1, 106.8)
- added REF**: MountingHole_2.2mm_M2_DIN965_Pad_TopBottom, Mounting Hole:MountingHole_2.2mm_M2_DIN965_Pad_TopBottom, F.Cu at (76.4, 47.9)
- added REF**: MountingHole_2.2mm_M2_DIN965_Pad_TopBottom, Mounting Hole:MountingHole_2.2mm_M2_DIN965_Pad_TopBottom, F.Cu at (183.0, 123.7)
- added REF**: MountingHole_2.2mm_M2_DIN965_Pad_TopBottom, Mounting Hole:MountingHole_2.2mm_M2_DIN965_Pad_TopBottom, F.Cu at (191.5, 118.0)
- added REF**: MountingHole_2.2mm_M2_DIN965_Pad_TopBottom, Mounting Hole:MountingHole_2.2mm_M2_DIN965_Pad_TopBottom, F.Cu at (116.4, 123.7)
- added REF**: MountingHole_2.2mm_M2_DIN965_Pad_TopBottom, Mounting Hole:MountingHole_2.2mm_M2_DIN965_Pad_TopBottom, F.Cu at (148.9, 96.8)
- added REF**: MountingHole_2.2mm_M2_DIN965_Pad_TopBottom, Mounting Hole:MountingHole_2.2mm_M2_DIN965_Pad_TopBottom, F.Cu at (172.0, 47.9)
- added REF**: MountingHole_2.2mm_M2_DIN965_Pad_TopBottom, Mounting Hole:MountingHole_2.2mm_M2_DIN965_Pad_TopBottom, F.Cu at (223.2, 118.0)
- added REF**: MountingHole_2.2mm_M2_DIN965_Pad_TopBottom, Mounting Hole:MountingHole_2.2mm_M2_DIN965_Pad_TopBottom, F.Cu at (76.4, 63.6)
- added REF**: MountingHole_2.2mm_M2_DIN965_Pad_TopBottom, Mounting Hole:MountingHole_2.2mm_M2_DIN965_Pad_TopBottom, F.Cu at (223.2, 62.0)
- added REF**: MountingHole_2.2mm_M2_DIN965_Pad_TopBottom, Mounting Hole:MountingHole_2.2mm_M2_DIN965_Pad_TopBottom, F.Cu at (92.3, 84.9)
- added REF**: MountingHole_2.2mm_M2_DIN965_Pad_TopBottom, Mounting Hole:MountingHole_2.2mm_M2_DIN965_Pad_TopBottom, F.Cu at (167.8, 80.2)
- added REF**: MountingHole_2.2mm_M2_DIN965_Pad_TopBottom, Mounting Hole:MountingHole_2.2mm_M2_DIN965_Pad_TopBottom, F.Cu at (92.3, 104.1)
Routing:
- net col0: track 193.1 -> 0.00 mm, vias 4 -> 0
- net col1: track 172.2 -> 0.00 mm, vias 4 -> 0
- net row2_r: track 163.5 -> 0.00 mm, vias 1 -> 0
- net GND: track 163.0 -> 0.00 mm, vias 2 -> 0
- net row1_r: track 162.9 -> 0.00 mm, vias 1 -> 0
- net row2: track 160.1 -> 0.00 mm, vias 1 -> 0
- net row0_r: track 159.2 -> 0.00 mm, vias 1 -> 0
- net row1: track 156.5 -> 0.00 mm, vias 1 -> 0
- net col2: track 154.6 -> 0.00 mm, vias 5 -> 0
- net col0_r: track 152.1 -> 0.00 mm, vias 4 -> 0
- net row0: track 151.8 -> 0.00 mm, vias 1 -> 0
- net col3: track 143.1 -> 0.00 mm, vias 5 -> 0
- net col2_r: track 140.3 -> 0.00 mm, vias 5 -> 0
- net col1_r: track 135.9 -> 0.00 mm, vias 6 -> 0
- net row3_r: track 134.0 -> 0.00 mm, vias 1 -> 0
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Other:
- board size 354 x 110 mm -> 153.7 x 110 mm
