File: sandevistan42/pcb/sandevistan44_right.kicad_pcb (KiCad board)
At the start: 2 copper layers, 354 x 110 mm, 114 parts, among them J1 TRRS, J2 TRRS, SW1 SW_PUSH, SW10 SW_PUSH, SW11 SW_PUSH, SW12 SW_PUSH, SW13 SW_PUSH, SW14 SW_PUSH, SW15 SW_PUSH, SW16 SW_PUSH, SW17 SW_PUSH, SW18 SW_PUSH, SW19 SW_PUSH, SW2 SW_PUSH, SW20 SW_PUSH, SW21 SW_PUSH, SW22 SW_PUSH, SW23 SW_PUSH, SW24 SW_PUSH, SW25 SW_PUSH, SW26 SW_PUSH, SW27 SW_PUSH, SW28 SW_PUSH, SW29 SW_PUSH, SW3 SW_PUSH, SW30 SW_PUSH, SW31 SW_PUSH, SW32 SW_PUSH, SW33 SW_PUSH, SW34 SW_PUSH, SW35 SW_PUSH, SW36 SW_PUSH, SW37 SW_PUSH, SW38 SW_PUSH, SW39 SW_PUSH, SW4 SW_PUSH, SW40 SW_PUSH, SW41 SW_PUSH, SW42 SW_PUSH, SW43 SW_PUSH, SW44 SW_PUSH, SW5 SW_PUSH, SW6 SW_PUSH, SW7 SW_PUSH, SW8 SW_PUSH, SW9 SW_PUSH, U1 ProMicro, U2 ProMicro

Commit message: Split pcbs into separate files and add plates
Parts:
- removed D1, D10, D11, D12, D13, D14, D15, D16, D17, D18, D19, D2, D20, D21, D22, D3, D4, D5, D6, D7, D8, D9: D, Library:TH 1N4148 Diode (long)
- removed DISP1: DFR0664, Library:DFR0664_2in_RGB_TFT_Display_3_standoff
- removed J1: TRRS, SJ2 35954A SMT TR:CUI_SJ2-35954A-SMT-TR
- removed the RESET at (179.6, 116.0)
- removed the Ref** at (123.0, 116.8)
- removed the Ref** at (71.5, 160.3)
- removed the Ref** at (127.1, 84.5)
- removed the Ref** at (104.0, 133.4)
- removed the Ref** at (31.5, 84.5)
- removed the Ref** at (138.1, 160.3)
- removed the Ref** at (47.5, 140.7)
- removed the Ref** at (47.4, 121.5)
- removed the Ref** at (31.5, 100.2)
- removed SW1, SW10, SW11, SW12, SW13, SW14, SW15, SW16, SW17, SW18, SW19, SW2, SW20, SW21, SW3, SW4, SW5, SW6, SW7, SW8, SW9: SW_PUSH, Library:SW_Hotswap_Kailh_Choc_V2_1.00u
- removed SW22: SW_PUSH, Library:SW_Hotswap_Kailh_Choc_V2_1.25u
- removed U1: ProMicro, marbastlib-xp-promicroish:Helios_AC
- added Ref**: Val**, Mounting Hole:MountingHole_2.2mm_M2_DIN965, F.Cu at (196.0, 89.0)
- added Ref**: Val**, Mounting Hole:MountingHole_2.2mm_M2_DIN965, F.Cu at (196.0, 108.2)
- moved D42 168.2 mm to (128.2, 55.4)
- moved D24 168.2 mm to (204.7, 63.6)
- moved D29 168.2 mm to (183.6, 60.8)
- moved D32 168.2 mm to (173.5, 57.7)
- moved D33 168.2 mm to (165.8, 59.4)
- moved D35 168.2 mm to (161.2, 55.5)
- moved D37 168.2 mm to (149.8, 56.9)
- moved D38 168.2 mm to (145.3, 57.1)
- moved D39 168.2 mm to (143.7, 54.3)
- moved D40 168.2 mm to (137.8, 56.2)
- moved D41 168.2 mm to (128.3, 59.4)
- moved D44 168.2 mm to (118.3, 56.8)
- moved J2 168.2 mm to (69.2, 75.4)
- moved MBIO1 168.2 mm to (86.8, 126.0)
- moved Ref** 168.2 mm to (95.0, 121.9)
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Routing:
- net col0: track 193.1 -> 0.00 mm, vias 4 -> 0
- net col1: track 172.2 -> 0.00 mm, vias 4 -> 0
- net row2: track 160.1 -> 0.00 mm, vias 1 -> 0
- net row1: track 156.5 -> 0.00 mm, vias 1 -> 0
- net col2: track 154.6 -> 0.00 mm, vias 5 -> 0
- net row0: track 151.8 -> 0.00 mm, vias 1 -> 0
- net col3: track 143.1 -> 0.00 mm, vias 5 -> 0
- net row3: track 130.6 -> 0.00 mm, vias 1 -> 0
- net GND: track 113.5 -> 0.00 mm, vias 6 -> 0
- net col4: track 113.3 -> 0.00 mm, vias 5 -> 0
- net Net-(D18-A): track 97.0 -> 0.00 mm, vias 2 -> 0
- net col5: track 95.9 -> 0.00 mm, vias 5 -> 0
- net Net-(D22-A): track 92.1 -> 0.00 mm, vias 2 -> 0
- net Net-(D14-A): track 87.3 -> 0.00 mm, vias 2 -> 0
- net Net-(D10-A): track 78.1 -> 0.00 mm, vias 2 -> 0
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Other:
- board size 354 x 110 mm -> 153.7 x 110 mm
